File: Collection/Collection.sch (KiCad schematic (older format))
At the start: 174 parts, among them U1A AD8668, U1A? AD8668, U1B AD8668, U1B? AD8668, U1C AD8668, U1C? AD8668, U1D AD8668, U1D? AD8668, U1D? LM1875, U1D? LM324, U1D? LM741

Commit message: Updated Schematic.
Parts:
- L?: value FlyBack_Pri_9Winds -> FlyBack_Pri_6-12(9)Winds
- L?: value FlyBack_SEC_47Winds_220V -> FlyBack_SEC_40-60(47)Winds_220V
- L?: value FlyBack_SEC_13Winds_-100V -> FlyBack_SEC_10-15(13)Winds_-100V
- L?: value FlyBack_Pri_2-3Winds_6.3VRMS -> FlyBack_SEC_2-3Winds_6.3VRMS
- L?: value FlyBack_Pri_1600Winds_Anode_8-12KV -> FlyBack_SEC_1600Winds_Anode_8-12KV
Changed lines of the file:
@@
 P 14750 2250
 F 0 "L?" H 14850 2350 50  0000 L CNN
-F 1 "FlyBack_Pri_9Winds" H 14850 2250 50  0000 L CNN
+F 1 "FlyBack_Pri_6-12(9)Winds" H 14850 2250 50  0000 L CNN
 F 2 "" H 14750 2250 50  0001 C CNN
 F 3 "~" H 14750 2250 50  0001 C CNN
@@
 P 14050 3500
 F 0 "L?" H 14000 3450 50  0000 R CNN
-F 1 "FlyBack_SEC_47Winds_220V" H 13900 3550 50  0000 R CNN
+F 1 "FlyBack_SEC_40-60(47)Winds_220V" H 13900 3550 50  0000 R CNN
 F 2 "" H 14050 3500 50  0001 C CNN
 F 3 "~" H 14050 3500 50  0001 C CNN
@@
 P 14050 3900
 F 0 "L?" H 14000 3800 50  0000 R CNN
-F 1 "FlyBack_SEC_13Winds_-100V" H 13950 3900 50  0000 R CNN
+F 1 "FlyBack_SEC_10-15(13)Winds_-100V" H 13950 3900 50  0000 R CNN
 F 2 "" H 14050 3900 50  0001 C CNN
 F 3 "~" H 14050 3900 50  0001 C CNN
@@
 P 14050 4300
 F 0 "L?" H 14000 4250 50  0000 R CNN
-F 1 "FlyBack_Pri_2-3Winds_6.3VRMS" H 13950 4350 50  0000 R CNN
+F 1 "FlyBack_SEC_2-3Winds_6.3VRMS" H 13950 4350 50  0000 R CNN
 F 2 "" H 14050 4300 50  0001 C CNN
 F 3 "~" H 14050 4300 50  0001 C CNN
@@
 P 14050 4700
 F 0 "L?" H 14200 4850 50  0000 R CNN
-F 1 "FlyBack_Pri_1600Winds_Anode_8-12KV" H 14000 4750 50  0000 R CNN
+F 1 "FlyBack_SEC_1600Winds_Anode_8-12KV" H 14000 4750 50  0000 R CNN
 F 2 "" H 14050 4700 50  0001 C CNN
 F 3 "~" H 14050 4700 50  0001 C CNN
